File: bicolor_ctrl/bicolor_ctrl.kicad_pcb (KiCad board)
At the start: 2 copper layers, 34.5 x 18.8 mm, 19 parts, among them J1 Conn_01x03_Pin, U1 LM393LVDR, U2 FDV304P, U3 FDV303N, U4 FDV303N

Commit message: Added branding
Other:
- board text added: "DNF Designs 2026"
Changed lines of the file:
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@@
+		)
+	)
+	(gr_text "DNF Designs 2026"
+		(at 98.5 72.25 0)
+		(layer "F.SilkS")
+		(effects
+			(font
+				(size 1 1)
+				(thickness 0.2)
+				(bold yes)
+			)
+			(justify left bottom)
 		)
 	)
