File: bicolor_ctrl/bicolor_ctrl.kicad_sch (KiCad schematic)
At the start: 19 parts, among them J1 Conn_01x03_Pin, U1 LM393LVDR, U2 FDV304P, U3 FDV303N, U4 FDV303N

Commit message: Added branding
Other:
- company: (none) -> DNF Designs
- title: (none) -> Bicolor LED Analog Controller
Changed lines of the file:
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@@
 	(generator_version "9.0")
 	(paper "A4")
+	(title_block
+		(title "Bicolor LED Analog Controller")
+		(date "2026-05-10")
+		(rev "RevA")
+		(company "DNF Designs")
+	)
 	(junction
 		(at 83.82 66.04)
